File: hardware/despertador.brd (EAGLE design)
At the start: 95 x 55 mm, 3 parts, among them U1 ATMEGA32U4-AU

Commit message: Add files via upload
Parts:
- removed U$1: DS3231, Microcontroladores:PDIP
- removed U1: ATMEGA32U4-AU, atmel:QFP44_10X10_0.80
- added C1, C2, C3: (no value), rcl:E2,5-6
- added IC1: MEGA8-P, atmel:DIL28-3
- added IC2: MAX702CPA, maxim:DIL08
- added R1: (no value), rcl:0207/10
- added SG1: B/C11L, buzzer:B/C11L
- added U$3: DS3231, Microcontroladores:PDIP
- added X1: (no value), con-molex:KK-156-2
- added X2: MINI-USB-32005-201, con-cypressindustries:32005-201
- U$2: value DISPLAY-OLED-128X64-I2C -> DISPLAY-OLED-128X32; device diy-modules:DISPLAY-OLED-128X64-I2C -> diy-modules:DISPLAY-OLED-128X32
- moved U$2 31.8 mm to (74.0, 7.56), turned to 0 degrees
Connections:
- removed net AVCC: U1.24, U1.44
- new net N$3: C3.+, IC1.10
- new net N$4: IC1.1, R1.1
- new net N$5: IC1.28, U$2.3, U$3.16
- new net N$6: IC2.7, U$3.4
- net GND: now also C1.-, C2.-, C3.-, IC1.22, IC1.8, IC2.3, SG1.2, U$3.13, X1.1; no longer U$1.13, U1.15, U1.23, U1.35, U1.43, U1.5
- net N$1: now also IC1.27, U$2.4, U$3.15; no longer U$1.16, U$2.3, U1.18
- net N$2: now also C2.+, IC1.9; no longer U$1.15, U$2.4, U1.19
- net VCC: now also C1.+, IC1.20, IC1.7, IC2.2, R1.2, SG1.1, U$3.2, X1.2; no longer U$1.2, U1.14, U1.2, U1.34
Routing:
- net VCC: track 91.6 -> 313.7 mm
- net GND: track 87.0 -> 236.4 mm
- net N$5: track 0.00 -> 65.5 mm
- net N$3: track 0.00 -> 61.1 mm
- net N$4: track 0.00 -> 53.5 mm
- net N$1: track 50.0 -> 82.8 mm, vias 1 -> 0
- net N$2: track 53.3 -> 79.9 mm
- net N$6: track 0.00 -> 25.6 mm
- net AVCC: track 14.2 -> 0.00 mm, vias 2 -> 0
