File: hardware/despertador.sch (EAGLE design)
At the start: 3 parts, among them U1 ATMEGA32U4-AU

Commit message: Add files via upload
Parts:
- removed U$1: DS3231, Microcontroladores:DS3231
- removed U1: ATMEGA32U4-AU, atmel:ATMEGA32U4-AU
- added C1, C2, C3: (no value), rcl:CPOL-EUE2.5-6
- added IC1: MEGA8-P, atmel:MEGA8-P
- added IC2: MAX702CPA, maxim:MAX702CPA
- added R1: (no value), rcl:R-US_0207/10
- added SG1: B/C11L, buzzer:B/C11L
- added U$3: DS3231, Microcontroladores:DS3231
- added X1: (no value), con-molex:KK-156-2
- added X2: MINI-USB-32005-201, con-cypressindustries:MINI-USB-32005-201
- U$2: value DISPLAY-OLED-128X64-I2C -> DISPLAY-OLED-128X32; device diy-modules:DISPLAY-OLED-128X64-I2C -> diy-modules:DISPLAY-OLED-128X32
Connections:
- new net N$3: C3.+, IC1.PB7(XTAL2/TOSC2)
- new net N$4: IC1.PC6(/RESET), R1.1
- new net N$5: IC1.PC5(ADC5/SCL), U$2.SCL, U$3.SCL
- new net N$6: IC2.RST, U$3./RST
- net GND: now also C1.-, C2.-, C3.-, IC1.GND, IC1.GND@1, IC2.GND, SG1.2, U$3.GND, X1-1.S; no longer U$1.GND, U1G$1.UGND
- net N$1: now also IC1.PC4(ADC4/SDA), U$2.SDA, U$3.SDA; no longer U$1.SCL, U$2.SCL, U1G$1.(OC0B/SCL/INT0)PD0
- net N$2: now also C2.+, IC1.PB6(XTAL1/TOSC1); no longer U$1.SDA, U$2.SDA, U1G$1.(SDA/INT1)PD1
- net VCC: now also C1.+, IC1.AVCC, IC1.VCC@1, IC2.VCC, R1.2, SG1.1, U$3.VCC, X1-2.S; no longer U$1.VCC, U1G$1.UVCC
Other:
- moved on the sheet: U$2
